File: Temperature_probe.kicad_sch (KiCad schematic)
At the start: 9 parts, among them IC5 MAX31865ATP+T, J3 Conn_01x04_Pin

Commit message: Layout Changes, MPN Added
Parts:
- C11: GPN GPC0402104-25 -> (none); MPN (none) -> GPC0402104-25
- SEL0, SEL1, SEL2, SEL3: now left out of the parts list
